File: uCM4.kicad_sch (KiCad schematic)
At the start: 30 parts, among them J1 Conn_01x03, J2 Ethernet, J3 Micro_SD_Card, J4 USB_B_Micro, SW1 SW_DIP_x01, SW2 SW_DIP_x01, U1 RT9742GGJ5, U2 74LVC1G07, U3 TPD4EUSB30

Commit message: Add jumper and start routing
Fill missing footprint assignment, most importantly, SMD jumper to
switch to RPIBOOT temporarily. This allows to flash eMMC, if present,
but still boot from default memory.
Parts:
- JP1: footprint (none) -> Special:Jumper
- SW1, SW2: footprint (none) -> Button_Switch_THT:SW_PUSH_6mm
Changed lines of the file:
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@@
     (property "Reference" "JP1" (id 0) (at 137.16 162.0478 0))
     (property "Value" "SolderJumper_2_Open" (id 1) (at 137.16 164.3465 0))
-    (property "Footprint" "" (id 2) (at 137.16 166.37 0)
+    (property "Footprint" "Special:Jumper" (id 2) (at 137.16 166.37 0)
       (effects (font (size 1.27 1.27)) hide)
     )
@@
       (effects (font (size 1.27 1.27)) (justify right))
     )
-    (property "Footprint" "" (id 2) (at 16.51 160.02 0)
+    (property "Footprint" "Button_Switch_THT:SW_PUSH_6mm" (id 2) (at 16.51 160.02 0)
       (effects (font (size 1.27 1.27)) hide)
     )
@@
     (property "Reference" "SW2" (id 0) (at 125.73 171.8268 0))
     (property "Value" "SW_DIP_x01" (id 1) (at 125.73 174.1255 0))
-    (property "Footprint" "" (id 2) (at 125.73 177.8 0)
+    (property "Footprint" "Button_Switch_THT:SW_PUSH_6mm" (id 2) (at 125.73 177.8 0)
       (effects (font (size 1.27 1.27)) hide)
     )
@@
     )
     (path "/debd560e-0565-4cbf-9569-5f25352bd66e"
-      (reference "JP1") (unit 1) (value "SolderJumper_2_Open") (footprint "")
+      (reference "JP1") (unit 1) (value "SolderJumper_2_Open") (footprint "Special:Jumper")
     )
     (path "/6e99bc10-5f29-45d8-a271-3de00e4eb307"
@@
     )
     (path "/53e986ab-59c5-4be6-a04f-f5936095ef65"
-      (reference "SW1") (unit 1) (value "SW_DIP_x01") (footprint "")
+      (reference "SW1") (unit 1) (value "SW_DIP_x01") (footprint "Button_Switch_THT:SW_PUSH_6mm")
     )
     (path "/311375dd-fa64-4cb4-aaf9-68277d25563b"
-      (reference "SW2") (unit 1) (value "SW_DIP_x01") (footprint "")
+      (reference "SW2") (unit 1) (value "SW_DIP_x01") (footprint "Button_Switch_THT:SW_PUSH_6mm")
     )
     (path "/76d915db-a75c-454e-b4b8-962461913747"

Commit message: Connect GNDs to ground
Was overlooked in high-speed connector.
Connections:
- net GND: now also Module1.107 (GND), Module1.108 (GND), Module1.113 (GND), Module1.114 (GND), Module1.119 (GND), Module1.120 (GND), Module1.125 (GND), Module1.126 (GND), Module1.131 (GND), Module1.132 (GND), Module1.137 (GND), Module1.138 (GND), Module1.144 (GND), Module1.150 (GND), Module1.155 (GND), Module1.156 (GND), Module1.161 (GND), Module1.162 (GND), Module1.167 (GND), Module1.168 (GND), Module1.173 (GND), Module1.174 (GND), Module1.179 (GND), Module1.180 (GND), Module1.185 (GND), Module1.186 (GND), Module1.191 (GND), Module1.192 (GND), Module1.197 (GND), Module1.198 (GND)
Changed lines of the file:
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@@
   (junction (at 186.69 143.51) (diameter 1.016) (color 0 0 0 0))
   (junction (at 186.69 151.13) (diameter 1.016) (color 0 0 0 0))
+  (junction (at 186.69 158.75) (diameter 1.016) (color 0 0 0 0))
   (junction (at 250.19 52.07) (diameter 1.016) (color 0 0 0 0))
   (junction (at 250.19 59.69) (diameter 1.016) (color 0 0 0 0))
@@
   (junction (at 250.19 143.51) (diameter 1.016) (color 0 0 0 0))
   (junction (at 250.19 151.13) (diameter 1.016) (color 0 0 0 0))
+  (junction (at 250.19 158.75) (diameter 1.016) (color 0 0 0 0))
   (junction (at 252.73 41.91) (diameter 1.016) (color 0 0 0 0))
   (junction (at 255.27 39.37) (diameter 1.016) (color 0 0 0 0))
@@
     (stroke (width 0) (type solid) (color 0 0 0 0))
   )
+  (wire (pts (xy 180.975 158.75) (xy 180.975 160.02))
+    (stroke (width 0) (type solid) (color 0 0 0 0))
+  )
   (wire (pts (xy 186.69 44.45) (xy 186.69 52.07))
     (stroke (width 0) (type solid) (color 0 0 0 0))
@@
     (stroke (width 0) (type solid) (color 0 0 0 0))
   )
+  (wire (pts (xy 186.69 158.75) (xy 180.975 158.75))
+    (stroke (width 0) (type solid) (color 0 0 0 0))
+  )
   (wire (pts (xy 186.69 158.75) (xy 187.96 158.75))
     (stroke (width 0) (type solid) (color 0 0 0 0))
@@
   )
   (wire (pts (xy 252.73 71.12) (xy 255.27 71.12))
+    (stroke (width 0) (type solid) (color 0 0 0 0))
+  )
+  (wire (pts (xy 254 158.75) (xy 250.19 158.75))
+    (stroke (width 0) (type solid) (color 0 0 0 0))
+  )
+  (wire (pts (xy 254 161.29) (xy 254 158.75))
     (stroke (width 0) (type solid) (color 0 0 0 0))
   )
@@
     )
     (property "Datasheet" "" (id 3) (at 175.26 55.88 0)
+      (effects (font (size 1.27 1.27)) hide)
+    )
+    (pin "1")
+  )
+  (symbol (lib_id "power:GND") (at 180.975 160.02 0) (unit 1)
+    (in_bom yes) (on_board yes)
+    (property "Reference" "#PWR0118" (id 0) (at 180.975 166.37 0)
+      (effects (font (size 1.27 1.27)) hide)
+    )
+    (property "Value" "GND" (id 1) (at 180.975 164.3444 0))
+    (property "Footprint" "" (id 2) (at 180.975 160.02 0)
+      (effects (font (size 1.27 1.27)) hide)
+    )
+    (property "Datasheet" "" (id 3) (at 180.975 160.02 0)
+      (effects (font (size 1.27 1.27)) hide)
+    )
+    (pin "1")
+  )
+  (symbol (lib_id "power:GND") (at 254 161.29 0) (unit 1)
+    (in_bom yes) (on_board yes)
+    (property "Reference" "#PWR?" (id 0) (at 254 167.64 0)
+      (effects (font (size 1.27 1.27)) hide)
+    )
+    (property "Value" "GND" (id 1) (at 254 165.6144 0))
+    (property "Footprint" "" (id 2) (at 254 161.29 0)
+      (effects (font (size 1.27 1.27)) hide)
+    )
+    (property "Datasheet" "" (id 3) (at 254 161.29 0)
       (effects (font (size 1.27 1.27)) hide)
     )
@@
       (reference "#PWR0117") (unit 1) (value "GND") (footprint "")
     )
+    (path "/86f273dc-9ac2-44d7-a286-4e038104eaf0"
+      (reference "#PWR0118") (unit 1) (value "GND") (footprint "")
+    )
+    (path "/d2bfec5e-83c4-402c-9a53-b4d343f1da79"
+      (reference "#PWR?") (unit 1) (value "GND") (footprint "")
+    )
     (path "/9f0bf6b6-f69e-4ba4-81d2-ef53481fe7fd"

Commit message: Attempt to fix shield of Eth
Just a rename from Shield to SH. Seems to be failed. But, who knows.
Changed lines of the file:
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@@
   (symbol (lib_id "power:GND") (at 254 161.29 0) (unit 1)
     (in_bom yes) (on_board yes)
-    (property "Reference" "#PWR?" (id 0) (at 254 167.64 0)
+    (property "Reference" "#PWR0119" (id 0) (at 254 167.64 0)
       (effects (font (size 1.27 1.27)) hide)
     )
@@
     )
     (path "/d2bfec5e-83c4-402c-9a53-b4d343f1da79"
-      (reference "#PWR?") (unit 1) (value "GND") (footprint "")
+      (reference "#PWR0119") (unit 1) (value "GND") (footprint "")
     )
     (path "/9f0bf6b6-f69e-4ba4-81d2-ef53481fe7fd"

Commit message: Connect power of 74* buffer
It was missing till now. Also update PCB to reflect changes.
Connections:
- net VCC is gone; now on net +3V3: U2.5 (VCC)
Changed lines of the file:
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@@
+    (stroke (width 0) (type solid) (color 0 0 0 0))
+  )
+  (wire (pts (xy 141.605 182.88) (xy 146.05 182.88))
+    (stroke (width 0) (type solid) (color 0 0 0 0))
+  )
+  (wire (pts (xy 141.605 186.055) (xy 141.605 182.88))
     (stroke (width 0) (type solid) (color 0 0 0 0))
   )
@@
     (stroke (width 0) (type solid) (color 0 0 0 0))
   )
+  (wire (pts (xy 151.13 182.88) (xy 161.29 182.88))
+    (stroke (width 0) (type solid) (color 0 0 0 0))
+  )
   (wire (pts (xy 154.94 66.04) (xy 154.94 77.47))
     (stroke (width 0) (type solid) (color 0 0 0 0))
@@
   )
   (wire (pts (xy 156.21 194.31) (xy 160.02 194.31))
+    (stroke (width 0) (type solid) (color 0 0 0 0))
+  )
+  (wire (pts (xy 161.29 170.18) (xy 161.29 182.88))
     (stroke (width 0) (type solid) (color 0 0 0 0))
   )
@@
     (pin "1")
   )
+  (symbol (lib_id "power:+3.3V") (at 161.29 170.18 0) (unit 1)
+    (in_bom yes) (on_board yes)
+    (property "Reference" "#PWR?" (id 0) (at 161.29 173.99 0)
+      (effects (font (size 1.27 1.27)) hide)
+    )
+    (property "Value" "+3.3V" (id 1) (at 161.29 166.6326 0))
+    (property "Footprint" "" (id 2) (at 161.29 170.18 0)
+      (effects (font (size 1.27 1.27)) hide)
+    )
+    (property "Datasheet" "" (id 3) (at 161.29 170.18 0)
+      (effects (font (size 1.27 1.27)) hide)
+    )
+    (pin "1")
+  )
   (symbol (lib_id "power:+3.3V") (at 167.64 186.69 0) (unit 1)
     (in_bom yes) (on_board yes)
@@
     )
     (property "Datasheet" "" (id 3) (at 133.35 181.61 0)
+      (effects (font (size 1.27 1.27)) hide)
+    )
+    (pin "1")
+  )
+  (symbol (lib_id "power:GND") (at 141.605 186.055 0) (unit 1)
+    (in_bom yes) (on_board yes)
+    (property "Reference" "#PWR0120" (id 0) (at 141.605 192.405 0)
+      (effects (font (size 1.27 1.27)) hide)
+    )
+    (property "Value" "GND" (id 1) (at 141.605 190.3794 0))
+    (property "Footprint" "" (id 2) (at 141.605 186.055 0)
+      (effects (font (size 1.27 1.27)) hide)
+    )
+    (property "Datasheet" "" (id 3) (at 141.605 186.055 0)
       (effects (font (size 1.27 1.27)) hide)
     )
@@
       (reference "#PWR0119") (unit 1) (value "GND") (footprint "")
     )
+    (path "/8799d311-7097-45c3-85cd-de251a859a4a"
+      (reference "#PWR0120") (unit 1) (value "GND") (footprint "")
+    )
+    (path "/1f46fb11-3632-4bab-bb42-fb8cbe7df91c"
+      (reference "#PWR?") (unit 1) (value "+3.3V") (footprint "")
+    )
     (path "/9f0bf6b6-f69e-4ba4-81d2-ef53481fe7fd"
